Commit message: refactor(描述): 优化仿真碰撞与动力学参数

File: src/rebotarm_description/urdf/dm/urdf/rebotarm_dm.urdf (robot description, URDF)
Before this commit: robot reBot_B601_DM_with_gripper, 10 links, 9 joints
Links:
- link base_link: geometry collision box size=0.14 0.2 0.08265; visual mesh filename=package://rebotarm_description/urdf/dm/meshes/base_link.STL
- link gripper_left: geometry collision box size=0.0929 0.08861 0.03921; visual mesh filename=package://rebotarm_description/urdf/dm/meshes/gripper_left.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
- link gripper_link: geometry collision box size=0.0775 0.18407 0.077; visual mesh filename=package://rebotarm_description/urdf/dm/meshes/gripper_link.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
- link gripper_right: geometry collision box size=0.0929 0.08861 0.03921; visual mesh filename=package://rebotarm_description/urdf/dm/meshes/gripper_right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
- link link1: geometry collision box size=0.08698 0.07725 0.09102; visual mesh filename=package://rebotarm_description/urdf/dm/meshes/link1.STL
- link link2: geometry collision box size=0.321 0.057 0.06735; visual mesh filename=package://rebotarm_description/urdf/dm/meshes/link2.STL
- link link3: geometry collision box size=0.29778 0.105 0.08025; visual mesh filename=package://rebotarm_description/urdf/dm/meshes/link3.STL
- link link4: geometry collision box size=0.14579 0.11591 0.06676; visual mesh filename=package://rebotarm_description/urdf/dm/meshes/link4.STL
- link link5: geometry collision box size=0.07 0.077 0.08004; visual mesh filename=package://rebotarm_description/urdf/dm/meshes/link5.STL
- link link6: geometry collision box size=0.0568 0.0568 0.0095; visual mesh filename=package://rebotarm_description/urdf/dm/meshes/link6.STL

File: src/rebotarm_description/urdf/rs/urdf/rebotarm_rs.urdf (robot description, URDF)
Before this commit: robot 00-arm-rs_asm-v3, 10 links, 9 joints
Links:
- link base_link: geometry collision box size=0.14 0.2 0.075; visual mesh filename=package://rebotarm_description/urdf/rs/meshes/base_link.STL
- link gripper_end: geometry collision box size=0.084 0.18407 0.0818; visual mesh filename=package://rebotarm_description/urdf/rs/meshes/cnc7.STL
- link gripper_left: geometry collision box size=0.03844 0.08861 0.09335; visual mesh filename=package://rebotarm_description/urdf/rs/meshes/cnc_left.STL
- link gripper_right: geometry collision box size=0.03844 0.08861 0.09335; visual mesh filename=package://rebotarm_description/urdf/rs/meshes/cnc_right.STL
- link link1: geometry collision box size=0.08645 0.0865 0.10778; visual mesh filename=package://rebotarm_description/urdf/rs/meshes/link1.STL
- link link2: geometry collision box size=0.32653 0.08812 0.0655; visual mesh filename=package://rebotarm_description/urdf/rs/meshes/cnc2.STL
- link link3: geometry collision box size=0.29381 0.12925 0.0865; visual mesh filename=package://rebotarm_description/urdf/rs/meshes/cnc3.STL
- link link4: geometry collision box size=0.15639 0.13144 0.0865; visual mesh filename=package://rebotarm_description/urdf/rs/meshes/cnc4.STL
- link link5: geometry collision box size=0.088 0.0818 0.1037; visual mesh filename=package://rebotarm_description/urdf/rs/meshes/cnc5.STL
- link link6: geometry collision box size=0.0568 0.0568 0.0095; visual mesh filename=package://rebotarm_description/urdf/rs/meshes/link6.STL
