Commit message: feat(仿真): 增加双模式控制与夹爪

File: src/rebotarm_bringup/urdf/rebotarm_controlled.urdf.xacro (robot description, xacro)
@@ -8,4 +8,5 @@
   <xacro:arg name="motor_enable_mask" default="0,0,0,0,0,0"/>
   <xacro:arg name="mujoco_headless" default="false"/>
+  <xacro:arg name="control_mode" default="position"/>
   <xacro:property name="model" value="$(arg model)"/>
   <xacro:property name="transport" value="$(arg transport)"/>
@@ -24,4 +25,5 @@
     hold_only="$(arg hold_only)"
     motor_enable_mask="$(arg motor_enable_mask)"
-    mujoco_headless="$(arg mujoco_headless)"/>
+    mujoco_headless="$(arg mujoco_headless)"
+    control_mode="$(arg control_mode)"/>
 </robot>

File: src/rebotarm_hardware/ros2_control/rebotarm.ros2_control.xacro (robot description, xacro)
@@ -2,5 +2,5 @@
 <robot xmlns:xacro="http://www.ros.org/wiki/xacro">
   <xacro:macro name="rebotarm_ros2_control"
-    params="model transport:=mock can_interface:=can0 allow_motor_enable:=false hold_only:=true motor_enable_mask:='0,0,0,0,0,0' rs_soft_start_ms:=1000 max_tracking_error:=0.2 mit_kp:='10,15,15,15,12,10' mit_kd:='0.3,0.3,0.3,0.4,0.3,0.3' mujoco_headless:=false">
+    params="model transport:=mock can_interface:=can0 allow_motor_enable:=false hold_only:=true motor_enable_mask:='0,0,0,0,0,0' rs_soft_start_ms:=1000 max_tracking_error:=0.2 mit_kp:='10,15,15,15,12,10' mit_kd:='0.3,0.3,0.3,0.4,0.3,0.3' mujoco_headless:=false control_mode:=position">
     <ros2_control name="RebotArmSystem" type="system">
       <hardware>
@@ -39,7 +39,7 @@
       </hardware>
       <joint name="joint1">
-        <command_interface name="position">
-          <param name="min">-2.8</param>
-          <param name="max">2.8</param>
+        <command_interface name="${'effort' if transport == 'mujoco' and control_mode == 'effort' else 'position'}">
+          <param name="min">${-36.0 if transport == 'mujoco' and control_mode == 'effort' else -2.8}</param>
+          <param name="max">${36.0 if transport == 'mujoco' and control_mode == 'effort' else 2.8}</param>
         </command_interface>
         <state_interface name="position"/>
@@ -48,7 +48,7 @@
       </joint>
       <joint name="joint2">
-        <command_interface name="position">
-          <param name="min">${-3.14 if model == 'dm' else 0.0}</param>
-          <param name="max">${0.0 if model == 'dm' else 3.14}</param>
+        <command_interface name="${'effort' if transport == 'mujoco' and control_mode == 'effort' else 'position'}">
+          <param name="min">${-36.0 if transport == 'mujoco' and control_mode == 'effort' else (-3.14 if model == 'dm' else 0.0)}</param>
+          <param name="max">${36.0 if transport == 'mujoco' and control_mode == 'effort' else (0.0 if model == 'dm' else 3.14)}</param>
         </command_interface>
         <state_interface name="position"/>
@@ -57,7 +57,7 @@
       </joint>
       <joint name="joint3">
-        <command_interface name="position">
-          <param name="min">${-3.14 if model == 'dm' else 0.0}</param>
-          <param name="max">${0.0 if model == 'dm' else 3.14}</param>
+        <command_interface name="${'effort' if transport == 'mujoco' and control_mode == 'effort' else 'position'}">
+          <param name="min">${-36.0 if transport == 'mujoco' and control_mode == 'effort' else (-3.14 if model == 'dm' else 0.0)}</param>
+          <param name="max">${36.0 if transport == 'mujoco' and control_mode == 'effort' else (0.0 if model == 'dm' else 3.14)}</param>
         </command_interface>
         <state_interface name="position"/>
@@ -66,7 +66,7 @@
       </joint>
       <joint name="joint4">
-        <command_interface name="position">
-          <param name="min">${-1.87 if model == 'dm' else -1.57}</param>
-          <param name="max">1.57</param>
+        <command_interface name="${'effort' if transport == 'mujoco' and control_mode == 'effort' else 'position'}">
+          <param name="min">${-14.0 if transport == 'mujoco' and control_mode == 'effort' else (-1.87 if model == 'dm' else -1.57)}</param>
+          <param name="max">${14.0 if transport == 'mujoco' and control_mode == 'effort' else 1.57}</param>
         </command_interface>
         <state_interface name="position"/>
@@ -75,7 +75,7 @@
       </joint>
       <joint name="joint5">
-        <command_interface name="position">
-          <param name="min">-1.57</param>
-          <param name="max">1.57</param>
+        <command_interface name="${'effort' if transport == 'mujoco' and control_mode == 'effort' else 'position'}">
+          <param name="min">${-14.0 if transport == 'mujoco' and control_mode == 'effort' else -1.57}</param>
+          <param name="max">${14.0 if transport == 'mujoco' and control_mode == 'effort' else 1.57}</param>
         </command_interface>
         <state_interface name="position"/>
@@ -84,7 +84,7 @@
       </joint>
       <joint name="joint6">
-        <command_interface name="position">
-          <param name="min">-3.14</param>
-          <param name="max">3.14</param>
+        <command_interface name="${'effort' if transport == 'mujoco' and control_mode == 'effort' else 'position'}">
+          <param name="min">${-14.0 if transport == 'mujoco' and control_mode == 'effort' else -3.14}</param>
+          <param name="max">${14.0 if transport == 'mujoco' and control_mode == 'effort' else 3.14}</param>
         </command_interface>
         <state_interface name="position"/>
@@ -92,4 +92,20 @@
         <state_interface name="effort"/>
       </joint>
+      <xacro:if value="${transport == 'mujoco'}">
+        <joint name="gripper_joint1">
+          <command_interface name="position">
+            <param name="min">0.0</param>
+            <param name="max">0.05</param>
+          </command_interface>
+          <state_interface name="position"/>
+          <state_interface name="velocity"/>
+          <state_interface name="effort"/>
+        </joint>
+        <joint name="gripper_joint2">
+          <state_interface name="position"/>
+          <state_interface name="velocity"/>
+          <state_interface name="effort"/>
+        </joint>
+      </xacro:if>
     </ros2_control>
   </xacro:macro>

Commit message: feat(仿真): 增加传感器与算法扩展接口

File: src/rebotarm_bringup/urdf/rebotarm_controlled.urdf.xacro (robot description, xacro)
@@ -9,4 +9,7 @@
   <xacro:arg name="mujoco_headless" default="false"/>
   <xacro:arg name="control_mode" default="position"/>
+  <xacro:arg name="sim_speed_factor" default="1.0"/>
+  <xacro:arg name="enable_ft_sensor" default="true"/>
+  <xacro:arg name="enable_camera" default="false"/>
   <xacro:property name="model" value="$(arg model)"/>
   <xacro:property name="transport" value="$(arg transport)"/>
@@ -18,4 +21,24 @@
   </xacro:if>
   <xacro:include filename="$(find rebotarm_hardware)/ros2_control/rebotarm.ros2_control.xacro"/>
+  <xacro:if value="${transport == 'mujoco'}">
+    <link name="wrist_camera_link"/>
+    <joint name="wrist_camera_joint" type="fixed">
+      <parent link="gripper_tcp"/>
+      <child link="wrist_camera_link"/>
+      <origin xyz="0 0 0.03" rpy="0 0 0"/>
+    </joint>
+    <link name="wrist_camera_optical_frame"/>
+    <joint name="wrist_camera_optical_joint" type="fixed">
+      <parent link="wrist_camera_link"/>
+      <child link="wrist_camera_optical_frame"/>
+      <origin xyz="0 0 0" rpy="-1.570796 0 -1.570796"/>
+    </joint>
+    <link name="wrist_camera_mujoco_frame"/>
+    <joint name="wrist_camera_mujoco_joint" type="fixed">
+      <parent link="wrist_camera_optical_frame"/>
+      <child link="wrist_camera_mujoco_frame"/>
+      <origin xyz="0 0 0" rpy="3.141593 0 0"/>
+    </joint>
+  </xacro:if>
   <xacro:rebotarm_ros2_control
     model="${model}"
@@ -26,4 +49,7 @@
     motor_enable_mask="$(arg motor_enable_mask)"
     mujoco_headless="$(arg mujoco_headless)"
-    control_mode="$(arg control_mode)"/>
+    control_mode="$(arg control_mode)"
+    sim_speed_factor="$(arg sim_speed_factor)"
+    enable_ft_sensor="$(arg enable_ft_sensor)"
+    enable_camera="$(arg enable_camera)"/>
 </robot>

File: src/rebotarm_hardware/ros2_control/rebotarm.ros2_control.xacro (robot description, xacro)
@@ -2,5 +2,5 @@
 <robot xmlns:xacro="http://www.ros.org/wiki/xacro">
   <xacro:macro name="rebotarm_ros2_control"
-    params="model transport:=mock can_interface:=can0 allow_motor_enable:=false hold_only:=true motor_enable_mask:='0,0,0,0,0,0' rs_soft_start_ms:=1000 max_tracking_error:=0.2 mit_kp:='10,15,15,15,12,10' mit_kd:='0.3,0.3,0.3,0.4,0.3,0.3' mujoco_headless:=false control_mode:=position">
+    params="model transport:=mock can_interface:=can0 allow_motor_enable:=false hold_only:=true motor_enable_mask:='0,0,0,0,0,0' rs_soft_start_ms:=1000 max_tracking_error:=0.2 mit_kp:='10,15,15,15,12,10' mit_kd:='0.3,0.3,0.3,0.4,0.3,0.3' mujoco_headless:=false control_mode:=position sim_speed_factor:=1.0 enable_ft_sensor:=true enable_camera:=false">
     <ros2_control name="RebotArmSystem" type="system">
       <hardware>
@@ -8,5 +8,5 @@
           <plugin>mujoco_ros2_control/MujocoSystemInterface</plugin>
           <param name="headless">${mujoco_headless}</param>
-          <param name="sim_speed_factor">1.0</param>
+          <param name="sim_speed_factor">${sim_speed_factor}</param>
         </xacro:if>
         <xacro:unless value="${transport == 'mujoco'}">
@@ -107,4 +107,25 @@
           <state_interface name="effort"/>
         </joint>
+        <xacro:if value="${enable_ft_sensor}">
+          <sensor name="wrist_fts">
+            <param name="frame_id">gripper_tcp</param>
+            <param name="mujoco_type">fts</param>
+            <param name="mujoco_sensor_name">wrist</param>
+            <state_interface name="force.x"/>
+            <state_interface name="force.y"/>
+            <state_interface name="force.z"/>
+            <state_interface name="torque.x"/>
+            <state_interface name="torque.y"/>
+            <state_interface name="torque.z"/>
+          </sensor>
+        </xacro:if>
+        <xacro:if value="${enable_camera}">
+          <sensor name="wrist_camera">
+            <param name="frame_name">wrist_camera_optical_frame</param>
+            <param name="info_topic">/wrist_camera/color/camera_info</param>
+            <param name="image_topic">/wrist_camera/color/image_raw</param>
+            <param name="depth_topic">/wrist_camera/aligned_depth_to_color/image_raw</param>
+          </sensor>
+        </xacro:if>
       </xacro:if>
     </ros2_control>
